File: iGEM.kicad_pcb (KiCad board)
At the start: 4 copper layers, 81.1 x 56.1 mm, 50 parts, among them IC1 TMCS1107A1BQDRQ1, IC2 TMCS1107A1BQDRQ1, IC3 MCP4642-502E_UN, J1 Conn_01x02, J2 Conn_01x02, J3 Conn_01x02, J4 Conn_01x03, M1 Fan, Q1 TIP122, Q2 TIP122, Q3 IRF4905, Q4 D44VH, Q5 IRF4905, Q6 D44VH, U1 ADC101C021CIMK, U2 ADC101C021CIMK, U3 PCA9536D, U4 ICL7667

Commit message: Changed to a single H-bridge for a single coil. Many parts changes. Addresses now configurable via pin header
Parts:
- removed C1, C11, C2, C3, C4, C5, C9: 0.1 uF, Capacitor_SMD:C_0805_2012Metric_Pad1.18x1.45mm_HandSolder
- removed C10, C6, C7, C8: 4.7 uF, Capacitor_Tantalum_SMD:CP_EIA-3528-21_Kemet-B_Pad1.50x2.35mm_HandSolder
- removed D1, D2: 1N4732A, Diode_THT:D_DO-41_SOD81_P10.16mm_Horizontal
- removed D3, D4: SB2060, Diode_THT:D_DO-201AD_P12.70mm_Horizontal
- removed F1: 15A, Fuse:Fuseholder_Blade_Mini_Keystone_3568
- removed H1, H2, H3, H4: MH, MountingHole:MountingHole_3.2mm_M3_DIN965_Pad
- removed HS1, HS2: Heatsink, Heatsink:Heatsink_AAVID_576802B03900G
- removed IC1, IC2: TMCS1107A1BQDRQ1, Package_SO:SOIC-8_3.9x4.9mm_P1.27mm
- removed IC3: MCP4642-502E_UN, Package_SO:MSOP-10_3x3mm_P0.5mm
- removed J1, J2: Conn_01x02, TerminalBlock:TerminalBlock_bornier-2_P5.08mm
- removed J3: Conn_01x02, 8PCV-02-006:8PCV02006
- removed J4: Conn_01x03, Connector_JST:JST_XH_B3B-XH-A_1x03_P2.50mm_Vertical
- removed M1: Fan, Connector_JST:JST_XH_B2B-XH-A_1x02_P2.50mm_Vertical
- removed Q1, Q2: TIP122, Package_TO_SOT_THT:TO-220-3_Vertical
- removed Q3, Q5: IRF4905, Package_TO_SOT_THT:TO-220-3_Vertical
- removed Q4, Q6: D44VH, Package_TO_SOT_THT:TO-220-3_Vertical
- removed R1, R2, R7, R8: 30 Ohm, Capacitor_SMD:C_0805_2012Metric_Pad1.18x1.45mm_HandSolder
- removed R10, R9: 4.7K, Resistor_SMD:R_0805_2012Metric_Pad1.20x1.40mm_HandSolder
- removed R3: 220 mOhm, TerminalBlock:TerminalBlock_bornier-2_P5.08mm
- removed R4: 3.3 Ohm, TerminalBlock:TerminalBlock_bornier-2_P5.08mm
- removed R5, R6: 10K, Capacitor_SMD:C_0805_2012Metric_Pad1.18x1.45mm_HandSolder
- removed U1, U2: ADC101C021CIMK, Package_TO_SOT_SMD:SOT-23-6
- removed U3: PCA9536D, Package_SO:SOIC-8_3.9x4.9mm_P1.27mm
- removed U4: ICL7667, Package_SO:SOIC-8_3.9x4.9mm_P1.27mm
Routing:
- net SDA: track 99.3 -> 0.00 mm, vias 1 -> 0
- net SCL: track 92.7 -> 0.00 mm, vias 1 -> 0
- net RHEO2_OUT: track 53.0 -> 0.00 mm
- net +5V: track 47.5 -> 0.00 mm, vias 12 -> 0
- net RHEO1_OUT: track 32.3 -> 0.00 mm
- net GND: track 31.9 -> 0.00 mm, vias 23 -> 0
- net Net-(R8-Pad2): track 30.5 -> 0.00 mm
- net Net-(R7-Pad1): track 28.8 -> 0.00 mm
- net PWM1: track 13.8 -> 0.00 mm
- net PWM2: track 9.67 -> 0.00 mm
- net Net-(Q2-Pad3): track 7.64 -> 0.00 mm
- net Net-(Q1-Pad3): track 7.36 -> 0.00 mm
- net Net-(IC1-Pad7): track 7.01 -> 0.00 mm
- net Net-(IC2-Pad7): track 6.67 -> 0.00 mm
- net RHEO2_IN: track 4.85 -> 0.00 mm
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- removed copper zone on In2.Cu, net +5V
- removed copper zone on In1.Cu, net GND
- removed copper zone on B.Cu, net Net-(D3-Pad1)
- removed copper zone on F.Cu, net Net-(D3-Pad1)
- removed copper zone on B.Cu, net Net-(D3-Pad2)
- removed copper zone on F.Cu, net Net-(D3-Pad2)
- removed copper zone on B.Cu, net Net-(D4-Pad1)
- removed copper zone on F.Cu, net Net-(D4-Pad1)
- removed copper zone on B.Cu, net Net-(D4-Pad2)
- removed copper zone on F.Cu, net Net-(D4-Pad2)
- removed copper zone on B.Cu, net Net-(F1-Pad1)
- removed copper zone on F.Cu, net Net-(F1-Pad1)
- removed copper zone on B.Cu, net Net-(HS1-Pad1)
- removed copper zone on F.Cu, net Net-(HS1-Pad1)
- removed copper zone on B.Cu, net Net-(HS2-Pad1)
- removed copper zone on F.Cu, net Net-(HS2-Pad1)
- removed copper zone on B.Cu, net Net-(Q4-Pad3)
- removed copper zone on F.Cu, net Net-(Q4-Pad3)
- removed copper zone on B.Cu, net Net-(Q6-Pad3)
- removed copper zone on F.Cu, net Net-(Q6-Pad3)
Other:
- board outline removed
- board text removed: "+"
- board text removed: "-"
- board text removed: "GND"
- board text removed: "Hopkins iGEM Constant Current Coil Driver Design by Sreenivas Eadara"
- board text removed: "SCL"
- board text removed: "SDA"

Commit message: Changes to improve thermals and layout
Parts:
- added C1: 0.1 uF, Capacitor_SMD:C_0805_2012Metric_Pad1.18x1.45mm_HandSolder, F.Cu at (109.0, 57.0)
- added C11: 0.1 uF, Capacitor_SMD:C_0805_2012Metric_Pad1.18x1.45mm_HandSolder, F.Cu at (99.0, 82.8)
- added C2: 0.1 uF, Capacitor_SMD:C_0805_2012Metric_Pad1.18x1.45mm_HandSolder, F.Cu at (100.2, 119.5)
- added C3: 0.1 uF, Capacitor_SMD:C_0805_2012Metric_Pad1.18x1.45mm_HandSolder, F.Cu at (111.8, 77.8)
- added C4: 0.1 uF, Capacitor_SMD:C_0805_2012Metric_Pad1.18x1.45mm_HandSolder, F.Cu at (94.8, 117.2)
- added C5: 0.1 uF, Capacitor_SMD:C_0805_2012Metric_Pad1.18x1.45mm_HandSolder, F.Cu at (70.2, 111.5)
- added C6: 0.1 uF, Capacitor_SMD:C_0805_2012Metric_Pad1.18x1.45mm_HandSolder, F.Cu at (138.8, 111.6)
- added C7: 4.7 uF, Capacitor_Tantalum_SMD:CP_EIA-3528-21_Kemet-B_Pad1.50x2.35mm_HandSolder, F.Cu at (95.5, 120.0)
- added C8: 0.1 uF, Capacitor_SMD:C_0805_2012Metric_Pad1.18x1.45mm_HandSolder, F.Cu at (107.0, 67.8)
- added C9: 10000 uF, Capacitor_THT:CP_Radial_D22.0mm_P10.00mm_SnapIn, F.Cu at (70.8, 82.0)
- added D1: 1N4732A, Diode_THT:D_DO-41_SOD81_P10.16mm_Horizontal, F.Cu at (99.5, 88.5)
- added D2: SB2060, Diode_THT:D_DO-201AD_P12.70mm_Horizontal, F.Cu at (85.3, 125.8)
- added D3: SB2060, Diode_THT:D_DO-201AD_P12.70mm_Horizontal, F.Cu at (72.2, 98.2)
- added D4: SB2060, Diode_THT:D_DO-201AD_P12.70mm_Horizontal, F.Cu at (136.3, 98.2)
- added D5: SB2060, Diode_THT:D_DO-201AD_P12.70mm_Horizontal, F.Cu at (123.5, 125.8)
- added D6: LED, LED_SMD:LED_0805_2012Metric_Pad1.15x1.40mm_HandSolder, F.Cu at (113.8, 49.2)
- added D7: 1N4732A, Diode_THT:D_DO-41_SOD81_P10.16mm_Horizontal, F.Cu at (114.5, 88.5)
- added D8: LED, LED_SMD:LED_0805_2012Metric_Pad1.15x1.40mm_HandSolder, F.Cu at (109.2, 49.2)
- added F1: 20A, Fuse:Fuseholder_Blade_Mini_Keystone_3568, F.Cu at (69.8, 58.0)
- added H1: MH, MountingHole:MountingHole_3.2mm_M3_DIN965_Pad, F.Cu at (142.0, 126.0)
- added H2: MH, MountingHole:MountingHole_3.2mm_M3_DIN965_Pad, F.Cu at (67.0, 51.0)
- added H3: MH, MountingHole:MountingHole_3.2mm_M3_DIN965_Pad, F.Cu at (142.0, 51.0)
- added H4: MH, MountingHole:MountingHole_3.2mm_M3_DIN965_Pad, F.Cu at (67.0, 126.0)
- added HS1: Heatsink, Heatsink:Heatsink_AAVID_576802B03900G, F.Cu at (102.6, 104.0)
- added HS2: Heatsink, Heatsink:Heatsink_AAVID_576802B03900G, F.Cu at (118.0, 104.0)
- added IC1: TMCS1107A1BQDRQ1, Package_SO:SOIC-8_3.9x4.9mm_P1.27mm, F.Cu at (102.8, 114.5)
- added IC2: MCP4642-502E_UN, MCP4642-502E_UN:SOP50P490X110-10N, F.Cu at (104.0, 80.2)
- added IC3: SN74LVC2G08IDCTRQ1, Package_SO:MSOP-8_3x3mm_P0.65mm, F.Cu at (111.0, 69.5)
- added J1: COIL, TerminalBlock:TerminalBlock_bornier-2_P5.08mm, F.Cu at (101.9, 125.8)
- added J2: Conn_01x03, Connector_PinHeader_2.54mm:PinHeader_1x03_P2.54mm_Vertical, F.Cu at (90.0, 114.7)
- added J3: Conn_01x02, 8PCV-02-006:8PCV02006, F.Cu at (80.3, 64.1)
- added J4: Conn_01x03, Connector_JST:JST_XH_B3B-XH-A_1x03_P2.50mm_Vertical, F.Cu at (119.5, 51.2)
- added J5: Conn_01x03, Connector_PinHeader_2.54mm:PinHeader_1x03_P2.54mm_Vertical, F.Cu at (103.5, 84.8)
- added J6: Conn_02x03_Odd_Even, Connector_PinHeader_2.54mm:PinHeader_2x03_P2.54mm_Vertical, F.Cu at (102.2, 50.0)
- added M1: Fan, Connector_JST:JST_XH_B2B-XH-A_1x02_P2.50mm_Vertical, F.Cu at (132.0, 51.2)
- added Q1: TIP122, Package_TO_SOT_THT:TO-220-3_Vertical, F.Cu at (99.5, 92.5)
- added Q2: IPD042P03L3GATMA1, Package_TO_SOT_SMD:TO-252-2, F.Cu at (81.5, 105.8)
- added Q3: IRL1404ZSTRLPBF, Package_TO_SOT_SMD:TO-263-2, F.Cu at (79.9, 116.8)
- added Q4: D44VH, Package_TO_SOT_THT:TO-220-3_Vertical, F.Cu at (97.1, 101.5)
- added Q5: IPD042P03L3GATMA1, Package_TO_SOT_SMD:TO-252-2, F.Cu at (127.1, 105.8)
- added Q6: TIP122, Package_TO_SOT_THT:TO-220-3_Vertical, F.Cu at (114.5, 92.5)
- added Q7: D44VH, Package_TO_SOT_THT:TO-220-3_Vertical, F.Cu at (112.5, 101.5)
- added Q8: IRL1404ZSTRLPBF, Package_TO_SOT_SMD:TO-263-2, F.Cu at (129.1, 115.8)
- added R1: 1K Ohm, Resistor_SMD:R_0805_2012Metric_Pad1.20x1.40mm_HandSolder, F.Cu at (98.0, 79.2)
- added R10: 4.7K, Resistor_SMD:R_0805_2012Metric_Pad1.20x1.40mm_HandSolder, F.Cu at (123.0, 56.2)
- added R2: 220 mOhm, TerminalBlock:TerminalBlock_bornier-2_P5.08mm, F.Cu at (90.9, 125.8)
- added R3: 1K Ohm, Resistor_SMD:R_0805_2012Metric_Pad1.20x1.40mm_HandSolder, F.Cu at (111.5, 60.5)
- added R4: 10K, Resistor_SMD:R_0805_2012Metric_Pad1.20x1.40mm_HandSolder, F.Cu at (111.5, 62.5)
- added R5: 1K Ohm, Resistor_SMD:R_0805_2012Metric_Pad1.20x1.40mm_HandSolder, F.Cu at (102.6, 77.2)
- added R6: 220 mOhm, TerminalBlock:TerminalBlock_bornier-2_P5.08mm, F.Cu at (112.9, 125.8)
- added R7: 1K Ohm, Resistor_SMD:R_0805_2012Metric_Pad1.20x1.40mm_HandSolder, F.Cu at (108.2, 52.5)
- added R9: 4.7K, Resistor_SMD:R_0805_2012Metric_Pad1.20x1.40mm_HandSolder, F.Cu at (118.5, 56.2)
- added U1: ADC101C021CIMK, Package_TO_SOT_SMD:SOT-23-6, F.Cu at (94.8, 113.5)
- added U2: ATtiny412-SS, Package_SO:SOIC-8_3.9x4.9mm_P1.27mm, F.Cu at (106.0, 61.5)
- added U3: SN74LVC1G04DBVR, digikey-footprints:SOT-753, F.Cu at (111.8, 74.8)
- added U4: FAN3268TMX, Package_SO:SOIC-8_3.9x4.9mm_P1.27mm, F.Cu at (70.9, 105.9)
- added U5: FAN3268TMX, Package_SO:SOIC-8_3.9x4.9mm_P1.27mm, F.Cu at (139.4, 105.8)
Routing:
- net ENABLE: track 0.00 -> 134.1 mm
- net DIR2: track 0.00 -> 120.2 mm, vias 0 -> 2
- net SDA: track 0.00 -> 117.7 mm, vias 0 -> 4
- net DIR1: track 0.00 -> 115.9 mm, vias 0 -> 2
- net SCL: track 0.00 -> 111.1 mm, vias 0 -> 4
- net +5V: track 0.00 -> 38.8 mm, vias 0 -> 61
- net GND: track 0.00 -> 29.0 mm, vias 0 -> 98
- net PWM2: track 0.00 -> 21.6 mm
- net RHEO2_OUT: track 0.00 -> 17.9 mm
- net PWM1: track 0.00 -> 17.0 mm
- net UPDI: track 0.00 -> 16.5 mm
- net RHEO1_OUT: track 0.00 -> 14.6 mm
- net FET4: track 0.00 -> 13.2 mm
- net FET1: track 0.00 -> 12.5 mm
- net Net-(D6-Pad1): track 0.00 -> 11.3 mm
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- added copper zone on B.Cu, net +5V
- added copper zone on F.Cu, net +5V
- added copper zone on In2.Cu, net +5V
- added copper zone on In3.Cu, net +5V
- added copper zone on B.Cu, net GND
- added copper zone on F.Cu, net GND
- added copper zone on In1.Cu, net GND
- added copper zone on In2.Cu, net GND
- added copper zone on In4.Cu, net GND
- added copper zone on B.Cu, net Net-(D2-Pad1)
- added copper zone on F.Cu, net Net-(D2-Pad1)
- added copper zone on In2.Cu, net Net-(D2-Pad1)
- added copper zone on B.Cu, net Net-(D3-Pad2)
- added copper zone on F.Cu, net Net-(D3-Pad2)
- added copper zone on In2.Cu, net Net-(D3-Pad2)
- added copper zone on B.Cu, net Net-(D4-Pad2)
- added copper zone on F.Cu, net Net-(D4-Pad2)
- added copper zone on In2.Cu, net Net-(D4-Pad2)
- added copper zone on B.Cu, net Net-(D5-Pad1)
- added copper zone on F.Cu, net Net-(D5-Pad1)
- added copper zone on In2.Cu, net Net-(D5-Pad1)
- added copper zone on B.Cu, net Net-(F1-Pad1)
- added copper zone on F.Cu, net Net-(F1-Pad1)
- added copper zone on In2.Cu, net Net-(F1-Pad1)
- added copper zone on B.Cu, net Net-(IC1-Pad1)
- added copper zone on F.Cu, net Net-(IC1-Pad1)
- added copper zone on In2.Cu, net Net-(IC1-Pad1)
- added copper zone on B.Cu, net Net-(Q1-Pad3)
- added copper zone on F.Cu, net Net-(Q1-Pad3)
- added copper zone on In2.Cu, net Net-(Q1-Pad3)
- added copper zone on B.Cu, net Net-(Q4-Pad3)
- added copper zone on In2.Cu, net Net-(Q4-Pad3)
- added copper zone on B.Cu, net Net-(Q6-Pad3)
- added copper zone on F.Cu, net Net-(Q6-Pad3)
- added copper zone on In2.Cu, net Net-(Q6-Pad3)
- added copper zone on B.Cu, net Net-(Q7-Pad3)
- added copper zone on F.Cu, net Net-(Q7-Pad3)
- added copper zone on In2.Cu, net Net-(Q7-Pad3)
Other:
- board outline added: 83 x 83 mm
- copper layers 4 -> 6
