File: iGEM-melty.kicad_pcb (KiCad board)
At the start: 4 copper layers, 98 x 98 mm, 64 parts, among them IC1 TMCS1107A1BQDRQ1, IC2 MCP4642-502E_UN, IC3 SN74LVC2G08IDCTRQ1, IC4 NLSX4373DR2G, J1 COIL, J2 Conn_01x03, J3 Conn_01x02, J4 Conn_01x04, J5 Conn_01x03, J6 Conn_02x03_Odd_Even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

Commit message: Replace out of stock Stemma QT header
Parts:
- G***: moved to B.Cu
- J4: footprint Connector_JST:JST_SH_SM04B-SRSS-TB_1x04-1MP_P1.00mm_Horizontal -> Connector_JST:JST_XH_B4B-XH-A_1x04_P2.50mm_Vertical
- moved D9 17.9 mm to (154.1, 57.8), turned to 180 degrees
- moved G*** 15.5 mm to (149.4, 71.3), turned to -90 degrees
- moved J4 6.81 mm to (130.0, 51.5)
- moved C12 3.09 mm to (128.5, 55.8)
- moved M1 2.70 mm to (148.8, 51.5), turned to 180 degrees
- moved IC4 2.16 mm to (123.8, 58.2)
- moved C13 2.05 mm to (128.5, 60.8)
- moved G*** 0.56 mm to (154.2, 66.0)
Routing:
- net VCC: track 9.57 -> 12.1 mm
- net SDA: track 84.3 -> 86.7 mm
- net GND: track 36.2 -> 33.8 mm, vias 120 -> 119
- net SCL: track 86.8 -> 87.9 mm
Other:
- board text added: "Coil Driver Hopkins iGEM Sreeni Eadara"
- board text added: "I2C"
- board text added: "SCL"
- board text added: "SDA"
- board text added: "VCC"
- board text removed: "Coil Driver - Hopkins iGEM Design by Sreenivas Eadara"
- board text removed: "STEMMA QT"

Commit message: miscellaneous improvements and cleanup
Parts:
- moved C5 9.13 mm to (66.1, 111.0), turned to 180 degrees
- moved U1 6.94 mm to (108.3, 123.3), turned to 0 degrees
- moved C7 4.30 mm to (108.4, 117.3), turned to 0 degrees
- moved C4 2.27 mm to (108.0, 120.3), turned to 0 degrees
- moved U4 2.16 mm to (68.0, 105.9), turned to -90 degrees
Routing:
- net DIR1: track 159.2 -> 140.8 mm
- net DIR2: track 142.8 -> 127.8 mm
- net Net-(IC1-Pad7): track 15.4 -> 5.88 mm
- net Net-(J2-Pad2): track 7.38 -> 15.5 mm
- net SDA: track 86.7 -> 93.3 mm
- net SCL: track 87.9 -> 93.9 mm
- net FET1: track 7.47 -> 12.5 mm
- net FET3: track 11.2 -> 6.50 mm
- net +5V: track 40.5 -> 43.1 mm, vias 76 -> 73
- net GND: track 33.8 -> 35.3 mm
- net ENABLE: track 169.7 -> 168.3 mm, vias 0 -> 2
- net PWM1: track 20.0 -> 21.4 mm
- net PWM2: track 19.5 -> 20.2 mm
- net VCC: track 12.1 -> 12.7 mm
- net Net-(IC3-Pad5): track 2.70 -> 3.30 mm
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